File: electronics/stepper.brd (EAGLE design)
At the start: 50.8 x 44.5 mm, 17 parts, among them J1 1-770969-0, J2 1-770968-0, J3 DF1BZ-8DP-2.5DSA, J4 S4B-XH-A, U1 ATMEGA328PB32-TQFP

Commit message: Finished stepper layout.
Routing:
- net N$5: track 4.38 -> 9.46 mm, vias 0 -> 2
- net GND: track 0.00 -> 2.17 mm, vias 0 -> 8
- net SDA: track 28.3 -> 30.0 mm
- net +12V: track 25.5 -> 24.8 mm
- added copper zone on layer 16, net GND
Other:
- board text added: "Magnetic Chess Stepper Driver KSU Eclub 2019 - 2020 Rev 1 Miranda Dodson"
